File: pwr_neg_bipolar.brd (EAGLE design)
At the start: 100 x 50 mm, 20 parts, among them T1 2SA1943

Commit message: latest
Parts:
- R2: value 10k -> 3k3
Changed lines of the file:
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@@
 <element name="R7" library="rcl" package="0922V" value="3K/3W" x="21.59" y="7.62" rot="R45"/>
 <element name="T1" library="transistor" package="TOP3V" value="2SA1943" x="75.8" y="6.5" rot="R180"/>
-<element name="R2" library="rcl" package="0411/12" value="10k" x="49.53" y="21.59" rot="R270"/>
+<element name="R2" library="rcl" package="0411/12" value="3k3" x="49.53" y="21.59" rot="R270"/>
 <element name="R8" library="rcl" package="0411/12" value="DNP1" x="59.69" y="21.59" rot="R270"/>
 <element name="C6" library="rcl" package="E7,5-16" value="1000uF 63V" x="66.04" y="38.1" rot="R180"/>
