File: pwr_neg_bipolar.sch (EAGLE design)
At the start: 20 parts, among them T1 2SA1943

Commit message: latest
Parts:
- R2: value 10k -> 3k3
Changed lines of the file:
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@@
 <part name="R7" library="rcl" deviceset="R-EU_" device="0922V" value="3K/3W"/>
 <part name="T1" library="transistor" deviceset="*-PNP-" device="TOP3V" value="2SA1943"/>
-<part name="R2" library="rcl" deviceset="R-EU_" device="0411/12" value="10k"/>
+<part name="R2" library="rcl" deviceset="R-EU_" device="0411/12" value="3k3"/>
 <part name="R8" library="rcl" deviceset="R-EU_" device="0411/12" value="DNP1"/>
 <part name="C6" library="rcl" deviceset="CPOL-EU" device="E7.5-16" value="1000uF 63V"/>
