File: pwr_pos_bipolar.brd (EAGLE design)
At the start: 100 x 50 mm, 20 parts

Commit message: ripple filter built and tested
Parts:
- R12: value DNP2 -> 22k
- R2: value 10k -> 22k
- R8: value DNP1 -> 2M2
- T2: value (none) -> BUX85
- U$11: value NPN-POWER -> ST13007
Changed lines of the file:
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@@
 <attribute name="MF" value="" x="10.16" y="25" size="1.778" layer="27" rot="R90" display="off"/>
 </element>
-<element name="R12" library="rcl" package="0411/12" value="DNP2" x="69.1" y="27.94" rot="R90"/>
-<element name="R2" library="rcl" package="0411/12" value="10k" x="57.15" y="27.94" rot="R90"/>
+<element name="R12" library="rcl" package="0411/12" value="22k" x="69.1" y="27.94" rot="R90"/>
+<element name="R2" library="rcl" package="0411/12" value="22k" x="57.15" y="27.94" rot="R90"/>
 <element name="R7" library="rcl" package="0922V" value="30K/3W" x="22.86" y="39.37" rot="R315"/>
-<element name="R8" library="rcl" package="0411/12" value="DNP1" x="50.8" y="27.94" rot="R90"/>
-<element name="T2" library="transistor" package="TO220V" value="" x="54.61" y="43.5"/>
+<element name="R8" library="rcl" package="0411/12" value="2M2" x="50.8" y="27.94" rot="R90"/>
+<element name="T2" library="transistor" package="TO220V" value="BUX85" x="54.61" y="43.5"/>
 <element name="U$1" library="Simplex-Heatsinks" package="SK456-60-3XM3L" value="SK456-60-3XM3L" x="54.61" y="46.99" rot="R180"/>
 <element name="U$2" library="Simplex-Enclosures" package="RN" value="RN_POWER" x="5.75" y="3.25"/>
@@
 <element name="U$10" library="Simplex-rlc" package="C_20G10" value="NICHICON_SNAPINØ20" x="89.83" y="24.13" rot="R270"/>
 <element name="R1" library="rcl" package="0411/12" value="DNP3" x="77.47" y="27.94" rot="R90"/>
-<element name="U$11" library="Simplex-DiscreteSemi" package="TOP3V_TO220" value="NPN-POWER" x="74.61" y="43.5"/>
+<element name="U$11" library="Simplex-DiscreteSemi" package="TOP3V_TO220" value="ST13007" x="74.61" y="43.5"/>
 </elements>
 <signals>

Commit message: latest
Parts:
- R2: value 22k -> 47k
Changed lines of the file:
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@@
 </element>
 <element name="R12" library="rcl" package="0411/12" value="22k" x="69.1" y="27.94" rot="R90"/>
-<element name="R2" library="rcl" package="0411/12" value="22k" x="57.15" y="27.94" rot="R90"/>
+<element name="R2" library="rcl" package="0411/12" value="47k" x="57.15" y="27.94" rot="R90"/>
 <element name="R7" library="rcl" package="0922V" value="30K/3W" x="22.86" y="39.37" rot="R315"/>
 <element name="R8" library="rcl" package="0411/12" value="2M2" x="50.8" y="27.94" rot="R90"/>

Commit message: build done
Parts:
- D1: value 1N4004 -> 1N4007
- R12: value 22k -> DNP
- R2: value 47k -> 10k
- R7: value 30K/3W -> 1M/3W
- R8: value 2M2 -> 3M3
Changed lines of the file:
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@@
 <attribute name="MF" value="" x="10.16" y="25" size="1.778" layer="27" rot="R90" display="off"/>
 </element>
-<element name="R12" library="rcl" package="0411/12" value="22k" x="69.1" y="27.94" rot="R90"/>
-<element name="R2" library="rcl" package="0411/12" value="47k" x="57.15" y="27.94" rot="R90"/>
-<element name="R7" library="rcl" package="0922V" value="30K/3W" x="22.86" y="39.37" rot="R315"/>
-<element name="R8" library="rcl" package="0411/12" value="2M2" x="50.8" y="27.94" rot="R90"/>
+<element name="R12" library="rcl" package="0411/12" value="DNP" x="69.1" y="27.94" rot="R90"/>
+<element name="R2" library="rcl" package="0411/12" value="10k" x="57.15" y="27.94" rot="R90"/>
+<element name="R7" library="rcl" package="0922V" value="1M/3W" x="22.86" y="39.37" rot="R315"/>
+<element name="R8" library="rcl" package="0411/12" value="3M3" x="50.8" y="27.94" rot="R90"/>
 <element name="T2" library="transistor" package="TO220V" value="BUX85" x="54.61" y="43.5"/>
 <element name="U$1" library="Simplex-Heatsinks" package="SK456-60-3XM3L" value="SK456-60-3XM3L" x="54.61" y="46.99" rot="R180"/>
@@
 <element name="U$5" library="Simplex-Connectors" package="M1_OFFSET" value="M1" x="96.52" y="12.7" rot="R90"/>
 <element name="U$6" library="Simplex-Connectors" package="M1_OFFSET" value="M1" x="96.52" y="36.83" rot="R90"/>
-<element name="D1" library="diode" package="DO41-10" value="1N4004" x="63.5" y="27.94" rot="R270"/>
+<element name="D1" library="diode" package="DO41-10" value="1N4007" x="63.5" y="27.94" rot="R270"/>
 <element name="U$7" library="Simplex-rlc" package="C_20G10" value="NICHICON_SNAPINØ20" x="34.29" y="30.48" rot="R180"/>
 <element name="U$8" library="Simplex-rlc" package="C_20G10" value="NICHICON_SNAPINØ20" x="34.29" y="10.16" rot="R180"/>
