File: pwr_pos_bipolar.sch (EAGLE design)
At the start: 20 parts

Commit message: ripple filter built and tested
Parts:
- R12: value DNP2 -> 22k
- R2: value 10k -> 22k
- R8: value DNP1 -> 2M2
- T2: value (none) -> BUX85
- U$11: value NPN-POWER -> ST13007
Changed lines of the file:
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@@
 <part name="B1" library="Simplex-DiscreteSemi" deviceset="DIOTEC_BC5000" device="" value="B250C5000"/>
 <part name="R7" library="rcl" deviceset="R-EU_" device="0922V" value="30K/3W"/>
-<part name="R2" library="rcl" deviceset="R-EU_" device="0411/12" value="10k"/>
-<part name="R8" library="rcl" deviceset="R-EU_" device="0411/12" value="DNP1"/>
-<part name="R12" library="rcl" deviceset="R-EU_" device="0411/12" value="DNP2"/>
+<part name="R2" library="rcl" deviceset="R-EU_" device="0411/12" value="22k"/>
+<part name="R8" library="rcl" deviceset="R-EU_" device="0411/12" value="2M2"/>
+<part name="R12" library="rcl" deviceset="R-EU_" device="0411/12" value="22k"/>
 <part name="U$1" library="Simplex-Heatsinks" deviceset="SK456-60-3XM3L" device=""/>
 <part name="U$2" library="Simplex-Enclosures" deviceset="RN_POWER" device=""/>
@@
 <part name="U$5" library="Simplex-Connectors" deviceset="M1" device=""/>
 <part name="U$6" library="Simplex-Connectors" deviceset="M1" device=""/>
-<part name="T2" library="transistor" deviceset="*-NPN-" device="TO220V"/>
+<part name="T2" library="transistor" deviceset="*-NPN-" device="TO220V" value="BUX85"/>
 <part name="D1" library="diode" deviceset="1N4004" device=""/>
 <part name="U$7" library="Simplex-rlc" deviceset="NICHICON_SNAPIN" device="Ø20"/>
@@
 <part name="U$10" library="Simplex-rlc" deviceset="NICHICON_SNAPIN" device="Ø20"/>
 <part name="R1" library="rcl" deviceset="R-EU_" device="0411/12" value="DNP3"/>
-<part name="U$11" library="Simplex-DiscreteSemi" deviceset="NPN-POWER" device=""/>
+<part name="U$11" library="Simplex-DiscreteSemi" deviceset="NPN-POWER" device="" value="ST13007"/>
 </parts>
 <sheets>
 <sheet>
-<description>Rusia Neagra MKII power pcb</description>
+<description>Power Assy - Positive bipolar</description>
 <plain>
 <text x="355.6" y="10.16" size="3.81" layer="97">01</text>
@@
 </nets>
 </sheet>
-<sheet>
-<description>Rusia Neagra MKII main point to point</description>
-<plain>
-</plain>
-<instances>
-</instances>
-<busses>
-</busses>
-<nets>
-</nets>
-</sheet>

Commit message: latest
Parts:
- R2: value 22k -> 47k
Changed lines of the file:
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@@
 <part name="B1" library="Simplex-DiscreteSemi" deviceset="DIOTEC_BC5000" device="" value="B250C5000"/>
 <part name="R7" library="rcl" deviceset="R-EU_" device="0922V" value="30K/3W"/>
-<part name="R2" library="rcl" deviceset="R-EU_" device="0411/12" value="22k"/>
+<part name="R2" library="rcl" deviceset="R-EU_" device="0411/12" value="47k"/>
 <part name="R8" library="rcl" deviceset="R-EU_" device="0411/12" value="2M2"/>
 <part name="R12" library="rcl" deviceset="R-EU_" device="0411/12" value="22k"/>

Commit message: build done
Parts:
- D1: value 1N4004 -> 1N4007
- R12: value 22k -> DNP
- R2: value 47k -> 10k
- R7: value 30K/3W -> 1M/3W
- R8: value 2M2 -> 3M3
Changed lines of the file:
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@@
 <part name="F4" library="fuse" deviceset="FUSE" device="SH35"/>
 <part name="B1" library="Simplex-DiscreteSemi" deviceset="DIOTEC_BC5000" device="" value="B250C5000"/>
-<part name="R7" library="rcl" deviceset="R-EU_" device="0922V" value="30K/3W"/>
-<part name="R2" library="rcl" deviceset="R-EU_" device="0411/12" value="47k"/>
-<part name="R8" library="rcl" deviceset="R-EU_" device="0411/12" value="2M2"/>
-<part name="R12" library="rcl" deviceset="R-EU_" device="0411/12" value="22k"/>
+<part name="R7" library="rcl" deviceset="R-EU_" device="0922V" value="1M/3W"/>
+<part name="R2" library="rcl" deviceset="R-EU_" device="0411/12" value="10k"/>
+<part name="R8" library="rcl" deviceset="R-EU_" device="0411/12" value="3M3"/>
+<part name="R12" library="rcl" deviceset="R-EU_" device="0411/12" value="DNP"/>
 <part name="U$1" library="Simplex-Heatsinks" deviceset="SK456-60-3XM3L" device=""/>
 <part name="U$2" library="Simplex-Enclosures" deviceset="RN_POWER" device=""/>
@@
 <part name="U$6" library="Simplex-Connectors" deviceset="M1" device=""/>
 <part name="T2" library="transistor" deviceset="*-NPN-" device="TO220V" value="BUX85"/>
-<part name="D1" library="diode" deviceset="1N4004" device=""/>
+<part name="D1" library="diode" deviceset="1N4004" device="" value="1N4007"/>
 <part name="U$7" library="Simplex-rlc" deviceset="NICHICON_SNAPIN" device="Ø20"/>
 <part name="U$8" library="Simplex-rlc" deviceset="NICHICON_SNAPIN" device="Ø20"/>
